Commit message: Rebase from 'release/humble/tiago_description'

File: ros2_control/ros2_control.urdf.xacro (robot description, xacro)
@@ -65,5 +65,5 @@
         <!-- wrist -->
         <xacro:ros2_control_wrist_rotational name="arm_5" reduction="1.0" offset="${arm_5_joint_offset}" />
-        <xacro:ros2_control_wrist_differential name_1="arm_6" name_2="arm_7"
+        <xacro:ros2_control_wrist_differential name="arm" number_1="6" number_2="7"
                                                act_reduction_1="-1.0" act_reduction_2="1.0"
                                                jnt_reduction_1="1.0" jnt_reduction_2="1.0"

File: urdf/arm/arm.ros2_control.xacro (robot description, xacro)
@@ -20,19 +20,6 @@
       <state_interface name="effort" />
     </joint>
-    <!-- @TODO transmissions for ros2 system -->
-    <!--
-    <transmission name="${name}_${number}_trans">
-      <plugin>transmission_interface/SimpleTransmission</plugin>
-      <actuator name="${name}_${number}_motor" role="actuator1">
-        <mechanicalReduction>${reduction}</mechanicalReduction>
-      </actuator>
-      <joint name="${name}_${number}_joint">
-        <offset>${offset}</offset>
-        <hardwareInterface>hardware_interface/PositionJointInterface</hardwareInterface>
-        <hardwareInterface>hardware_interface/EffortJointInterface</hardwareInterface>
-        <hardwareInterface>hardware_interface/JointStateInterface</hardwareInterface>
-      </joint>
-    </transmission>
-    -->
+    <xacro:include filename="$(find tiago_description)/urdf/arm/arm.transmission.xacro" />
+    <xacro:arm_simple_transmission name="${name}" reduction="${reduction}" offset_value="${offset}"/>
   </xacro:macro>
 </robot>

File: urdf/arm/arm.transmission.xacro (robot description, xacro)
@@ -13,16 +13,12 @@
  -->
 <robot xmlns:xacro="http://ros.org/wiki/xacro">
-  <xacro:macro name="arm_simple_transmission" params="name number reduction offset_value" >
-    <transmission name="${name}_${number}_trans">
+  <xacro:macro name="arm_simple_transmission" params="name reduction offset_value" >
+    <transmission name="${name}_trans">
       <plugin>transmission_interface/SimpleTransmission</plugin>
-      <actuator name="${name}_${number}_motor"  role="actuator1">
-        <mechanicalReduction>${reduction}</mechanicalReduction>
-      </actuator>
-      <joint name="${name}_${number}_joint" role="joint1">
+      <actuator name="${name}_motor"  role="actuator1"/>
+      <joint name="${name}_joint" role="joint1">
+        <mechanical_reduction>${reduction}</mechanical_reduction>
         <offset>${offset_value}</offset>
-        <hardwareInterface>hardware_interface/PositionJointInterface</hardwareInterface>
-        <hardwareInterface>hardware_interface/EffortJointInterface</hardwareInterface>
-        <hardwareInterface>hardware_interface/JointStateInterface</hardwareInterface>
-      </joint>
+     </joint>
     </transmission>
   </xacro:macro>

File: urdf/arm/arm.urdf.xacro (robot description, xacro)
@@ -256,9 +256,4 @@
         <origin xyz="0 0 ${reflect * tool_link_z_offset}" rpy="${90.0 * deg_to_rad} ${reflect * -90.0 * deg_to_rad} ${180 * deg_to_rad}" />
     </joint>
-    <!-- extensions -->
-    <xacro:arm_simple_transmission name="${name}" number="1" reduction="1.0" offset_value="${arm_1_offset}"/>
-    <xacro:arm_simple_transmission name="${name}" number="2" reduction="1.0" offset_value="${arm_2_offset}"/>
-    <xacro:arm_simple_transmission name="${name}" number="3" reduction="1.0" offset_value="${arm_3_offset}"/>
-    <xacro:arm_simple_transmission name="${name}" number="4" reduction="1.0" offset_value="${arm_4_offset}"/>
   </xacro:macro>
 </robot>

File: urdf/arm/wrist.ros2_control.xacro (robot description, xacro)
@@ -20,23 +20,10 @@
       <state_interface name="effort" />
     </joint>
-    <!-- @TODO transmissions for ros2 system -->
-    <!--
-    <transmission name="${name}_${number}_trans">
-      <plugin>transmission_interface/SimpleTransmission</plugin>
-      <actuator name="${name}_${number}_motor" role="actuator1">
-        <mechanicalReduction>${reduction}</mechanicalReduction>
-      </actuator>
-      <joint name="${name}_${number}_joint">
-        <offset>${offset}</offset>
-        <hardwareInterface>hardware_interface/JointStateInterface</hardwareInterface>
-        <hardwareInterface>hardware_interface/PositionJointInterface</hardwareInterface>
-        <hardwareInterface>hardware_interface/EffortJointInterface</hardwareInterface>
-      </joint>
-    </transmission>
-    -->
+    <xacro:include filename="$(find tiago_description)/urdf/arm/wrist.transmission.xacro" />
+    <xacro:wrist_simple_transmission name="${name}" reduction="${reduction}" offset="${offset}"/>
   </xacro:macro>
   <xacro:macro name="ros2_control_wrist_differential"
-               params="name_1 name_2 act_reduction_1 act_reduction_2 jnt_reduction_1 jnt_reduction_2 number_1_offset number_2_offset" >
-    <joint name="${name_1}_joint">
+               params="name number_1 number_2 act_reduction_1 act_reduction_2 jnt_reduction_1 jnt_reduction_2 number_1_offset number_2_offset" >
+    <joint name="${name}_${number_1}_joint">
       <command_interface name="position" />
       <state_interface name="position" />
@@ -44,5 +31,5 @@
       <state_interface name="effort" />
     </joint>
-    <joint name="${name_2}_joint">
+    <joint name="${name}_${number_2}_joint">
       <command_interface name="position" />
       <state_interface name="position" />
@@ -50,32 +37,10 @@
       <state_interface name="effort" />
     </joint>
-    <!-- @TODO transmissions for ros2 system -->
-    <!--
-    <transmission name="${name1}_${name2}_wrist_trans">
-      <plugin>transmission_interface/DifferentialTransmission</plugin>
-      <actuator name="${name_1}_motor" role="actuator1">
-        <mechanicalReduction>${act_reduction_1}</mechanicalReduction>
-      </actuator>
-      <actuator name="${name_2}_motor" role="actuator2">
-        <mechanicalReduction>${act_reduction_2}</mechanicalReduction>
-      </actuator>
-      <joint name="${name_1}_joint" role="joint1">
-        <offset>${number_1_offset}</offset>
-        <mechanicalReduction>${jnt_reduction_1}</mechanicalReduction>
-        <hardwareInterface>hardware_interface/JointStateInterface</hardwareInterface>
-        <hardwareInterface>hardware_interface/PositionJointInterface</hardwareInterface>
-        <hardwareInterface>hardware_interface/EffortJointInterface</hardwareInterface>
-        <ignoreTransmissionAbsoluteEncoder>1</ignoreTransmissionAbsoluteEncoder>
-      </joint>
-      <joint name="${name_2}_joint" role="joint2">
-        <offset>${number_2_offset}</offset>
-        <mechanicalReduction>${jnt_reduction_2}</mechanicalReduction>
-        <hardwareInterface>hardware_interface/JointStateInterface</hardwareInterface>
-        <hardwareInterface>hardware_interface/PositionJointInterface</hardwareInterface>
-        <hardwareInterface>hardware_interface/EffortJointInterface</hardwareInterface>
-        <ignoreTransmissionAbsoluteEncoder>1</ignoreTransmissionAbsoluteEncoder>
-      </joint>
-    </transmission>
-    -->
+    <xacro:include filename="$(find tiago_description)/urdf/arm/wrist.transmission.xacro" />
+    <xacro:wrist_differential_transmission
+      name="${name}" number_1="${number_1}" number_2="${number_2}"
+      act_reduction_1="${act_reduction_1}" act_reduction_2="${act_reduction_2}"
+      jnt_reduction_1="${jnt_reduction_1}" jnt_reduction_2="${jnt_reduction_2}"
+      number_1_offset="${number_1_offset}" number_2_offset="${number_2_offset}"/>
   </xacro:macro>
 </robot>

File: urdf/arm/wrist.transmission.xacro (robot description, xacro)
@@ -13,15 +13,11 @@
  -->
 <robot xmlns:xacro="http://ros.org/wiki/xacro">
-  <xacro:macro name="wrist_simple_transmission" params="name number reduction offset" >
-    <transmission name="${name}_${number}_trans">
+  <xacro:macro name="wrist_simple_transmission" params="name reduction offset" >
+    <transmission name="${name}_trans">
       <plugin>transmission_interface/SimpleTransmission</plugin>
-      <actuator name="${name}_${number}_motor"  role="actuator1">
-        <mechanicalReduction>${reduction}</mechanicalReduction>
-      </actuator>
-      <joint name="${name}_${number}_joint" role="joint1">
+      <actuator name="${name}_motor"  role="actuator1"/>
+      <joint name="${name}_joint" role="joint1">
+        <mechanical_reduction>${reduction}</mechanical_reduction>
         <offset>${offset}</offset>
-        <hardwareInterface>hardware_interface/JointStateInterface</hardwareInterface>
-        <hardwareInterface>hardware_interface/PositionJointInterface</hardwareInterface>
-        <hardwareInterface>hardware_interface/EffortJointInterface</hardwareInterface>
       </joint>
     </transmission>
@@ -29,27 +25,19 @@
   <xacro:macro name="wrist_differential_transmission"
                params="name number_1 number_2 act_reduction_1 act_reduction_2 jnt_reduction_1 jnt_reduction_2 number_1_offset number_2_offset" >
-  <transmission name="${name}_wrist_trans">
+  <transmission name="${name}_${number_1}_${name}_${number_2}_wrist_trans">
       <plugin>transmission_interface/DifferentialTransmission</plugin>
       <actuator name="${name}_${number_1}_motor" role="actuator1">
-        <mechanicalReduction>${act_reduction_1}</mechanicalReduction>
+      <mechanical_reduction>${act_reduction_1}</mechanical_reduction>
       </actuator>
       <actuator name="${name}_${number_2}_motor" role="actuator2">
-        <mechanicalReduction>${act_reduction_2}</mechanicalReduction>
+        <mechanical_reduction>${act_reduction_2}</mechanical_reduction>
       </actuator>
       <joint name="${name}_${number_1}_joint" role="joint1">
+        <mechanical_reduction>${jnt_reduction_1}</mechanical_reduction>
         <offset>${number_1_offset}</offset>
-        <mechanicalReduction>${jnt_reduction_1}</mechanicalReduction>
-        <hardwareInterface>hardware_interface/JointStateInterface</hardwareInterface>
-        <hardwareInterface>hardware_interface/PositionJointInterface</hardwareInterface>
-        <hardwareInterface>hardware_interface/EffortJointInterface</hardwareInterface>
-        <ignoreTransmissionAbsoluteEncoder>1</ignoreTransmissionAbsoluteEncoder>
       </joint>
       <joint name="${name}_${number_2}_joint" role="joint2">
+        <mechanical_reduction>${jnt_reduction_2}</mechanical_reduction>
         <offset>${number_2_offset}</offset>
-        <mechanicalReduction>${jnt_reduction_2}</mechanicalReduction>
-        <hardwareInterface>hardware_interface/JointStateInterface</hardwareInterface>
-        <hardwareInterface>hardware_interface/PositionJointInterface</hardwareInterface>
-        <hardwareInterface>hardware_interface/EffortJointInterface</hardwareInterface>
-        <ignoreTransmissionAbsoluteEncoder>1</ignoreTransmissionAbsoluteEncoder>
       </joint>
     </transmission>

File: urdf/arm/wrist.urdf.xacro (robot description, xacro)
@@ -171,10 +171,4 @@
         <provideFeedback>1</provideFeedback>
     </gazebo>
-    <!-- extensions -->
-    <xacro:wrist_simple_transmission name="${name}" number="5" reduction="1.0" offset="${arm_5_offset}"/>
-    <xacro:wrist_differential_transmission name="${name}" number_1="6" number_2="7"
-                                                act_reduction_1="-1.0" act_reduction_2="1.0"
-                                                jnt_reduction_1="1.0" jnt_reduction_2="${-reflect}"
-                                                number_1_offset="${arm_6_offset}" number_2_offset="${arm_7_offset}"/>
   </xacro:macro>
 </robot>

File: urdf/head/head.ros2_control.xacro (robot description, xacro)
@@ -20,18 +20,6 @@
       <state_interface name="effort" />
     </joint>
-    <!-- @TODO transmissions for ros2 system -->
-    <!--
-    <transmission name="${name}_trans">
-      <plugin>transmission_interface/SimpleTransmission</plugin>
-      <actuator name="${name}_motor" role="actuator1">
-        <mechanicalReduction>${reduction}</mechanicalReduction>
-      </actuator>
-      <joint name="${name}_joint">
-        <offset>${offset_value}</offset>
-        <hardwareInterface>hardware_interface/PositionJointInterface</hardwareInterface>
-        <hardwareInterface>hardware_interface/JointStateInterface</hardwareInterface>
-      </joint>
-    </transmission>
-    -->
+    <xacro:include filename="$(find tiago_description)/urdf/head/head.transmission.xacro" />
+    <xacro:head_transmission name="${name}" reduction="${reduction}" offset_value="${offset}"/>
   </xacro:macro>
 </robot>

File: urdf/head/head.transmission.xacro (robot description, xacro)
@@ -16,11 +16,8 @@
     <transmission name="${name}_trans">
       <plugin>transmission_interface/SimpleTransmission</plugin>
-      <actuator name="${name}_motor"  role="actuator1">
-        <mechanicalReduction>${reduction}</mechanicalReduction>
-      </actuator>
+      <actuator name="${name}_motor"  role="actuator1"/>
       <joint name="${name}_joint"  role="joint1">
         <offset>${offset_value}</offset>
-        <hardwareInterface>hardware_interface/JointStateInterface</hardwareInterface>
-        <hardwareInterface>hardware_interface/PositionJointInterface</hardwareInterface>
+        <mechanical_reduction>${reduction}</mechanical_reduction>
       </joint>
     </transmission>

File: urdf/torso/torso.ros2_control.xacro (robot description, xacro)
@@ -20,17 +20,6 @@
       <state_interface name="effort" />
     </joint>
-    <!-- @TODO transmissions for ros2 system -->
-    <!--
-    <transmission name="${name}_trans">
-      <plugin>transmission_interface/SimpleTransmission</plugin>
-      <actuator name="${name}_motor" role="actuator1">
-        <mechanicalReduction>${reduction}</mechanicalReduction>
-      </actuator>
-      <joint name="${name}_joint">
-        <hardwareInterface>hardware_interface/PositionJointInterface</hardwareInterface>
-        <hardwareInterface>hardware_interface/JointStateInterface</hardwareInterface>
-      </joint>
-    </transmission>
-    -->
+    <xacro:include filename="$(find tiago_description)/urdf/torso/torso.transmission.xacro" />
+    <xacro:torso_simple_transmission name="${name}" reduction="${reduction}" />
   </xacro:macro>
 </robot>

File: urdf/torso/torso.transmission.xacro (robot description, xacro)
@@ -16,10 +16,7 @@
     <transmission name="${name}_trans">
       <plugin>transmission_interface/SimpleTransmission</plugin>
-      <actuator name="${name}_motor" role="actuator1">
-        <mechanicalReduction>${reduction}</mechanicalReduction>
-      </actuator>
+      <actuator name="${name}_motor" role="actuator1"/>
       <joint name="${name}_joint" role="joint1">
-        <hardwareInterface>hardware_interface/PositionJointInterface</hardwareInterface>
-        <hardwareInterface>hardware_interface/JointStateInterface</hardwareInterface>
+        <mechanical_reduction>${reduction}</mechanical_reduction>
       </joint>
     </transmission>
