Commit message: Imported upstream version '4.0.3' of 'upstream'

File: tiago_description/ros2_control/transmissions.urdf.xacro (robot description, xacro)
@@ -1,5 +1,5 @@
 <?xml version="1.0"?>
 <!--
-  Copyright (c) 2022 PAL Robotics S.L. All rights reserved.
+  Copyright (c) 2023 PAL Robotics S.L. All rights reserved.
   Licensed under the Apache License, Version 2.0 (the "License");
   you may not use this file except in compliance with the License.
@@ -13,5 +13,5 @@
  -->
 <robot xmlns:xacro="http://ros.org/wiki/xacro">
-  <xacro:macro name="wrist_simple_transmission" params="name reduction offset" >
+  <xacro:macro name="tiago_simple_transmission" params="name reduction:=1.0 offset_value:=0.0" >
     <transmission name="${name}_trans">
       <plugin>transmission_interface/SimpleTransmission</plugin>
@@ -19,9 +19,9 @@
       <joint name="${name}_joint" role="joint1">
         <mechanical_reduction>${reduction}</mechanical_reduction>
-        <offset>${offset}</offset>
-      </joint>
+        <offset>${offset_value}</offset>
+     </joint>
     </transmission>
   </xacro:macro>
-  <xacro:macro name="wrist_differential_transmission"
+  <xacro:macro name="tiago_differential_transmission"
                params="name number_1 number_2 act_reduction_1 act_reduction_2 jnt_reduction_1 jnt_reduction_2 number_1_offset number_2_offset" >
   <transmission name="${name}_${number_1}_${name}_${number_2}_wrist_trans">

File: tiago_description/urdf/arm/arm.ros2_control.xacro (robot description, xacro)
@@ -20,6 +20,6 @@
       <state_interface name="effort" />
     </joint>
-    <xacro:include filename="$(find tiago_description)/urdf/arm/arm.transmission.xacro" />
-    <xacro:arm_simple_transmission name="${name}" reduction="${reduction}" offset_value="${offset}"/>
+<xacro:include filename="$(find tiago_description)/ros2_control/transmissions.urdf.xacro" />
+<xacro:tiago_simple_transmission name="${name}" reduction="${reduction}" offset_value="${offset}" />
   </xacro:macro>
 </robot>

File: tiago_description/urdf/arm/arm.urdf.xacro (robot description, xacro)
@@ -16,5 +16,4 @@
   <xacro:include filename="$(find tiago_description)/urdf/deg_to_rad.xacro" />
   <xacro:include filename="$(find tiago_description)/urdf/arm/wrist.urdf.xacro" />
-  <xacro:include filename="$(find tiago_description)/urdf/arm/arm.transmission.xacro" />
   <!--Constant parameters-->
   <xacro:property name="arm_friction"       value="1.0" />

File: tiago_description/urdf/arm/wrist.ros2_control.xacro (robot description, xacro)
@@ -20,6 +20,6 @@
       <state_interface name="effort" />
     </joint>
-    <xacro:include filename="$(find tiago_description)/urdf/arm/wrist.transmission.xacro" />
-    <xacro:wrist_simple_transmission name="${name}" reduction="${reduction}" offset="${offset}"/>
+    <xacro:include filename="$(find tiago_description)/ros2_control/transmissions.urdf.xacro" />
+    <xacro:tiago_simple_transmission name="${name}" reduction="${reduction}" offset_value="${offset}" />
   </xacro:macro>
   <xacro:macro name="ros2_control_wrist_differential"
@@ -37,6 +37,6 @@
       <state_interface name="effort" />
     </joint>
-    <xacro:include filename="$(find tiago_description)/urdf/arm/wrist.transmission.xacro" />
-    <xacro:wrist_differential_transmission
+    <xacro:include filename="$(find tiago_description)/ros2_control/transmissions.urdf.xacro" />
+    <xacro:tiago_differential_transmission
       name="${name}" number_1="${number_1}" number_2="${number_2}"
       act_reduction_1="${act_reduction_1}" act_reduction_2="${act_reduction_2}"

File: tiago_description/urdf/arm/wrist.urdf.xacro (robot description, xacro)
@@ -15,5 +15,4 @@
   <!--File includes-->
   <xacro:include filename="$(find tiago_description)/urdf/deg_to_rad.xacro" />
-  <xacro:include filename="$(find tiago_description)/urdf/arm/wrist.transmission.xacro" />
   <!--Constant parameters-->
   <xacro:property name="wrist_friction"       value="1.0" />

File: tiago_description/urdf/head/head.ros2_control.xacro (robot description, xacro)
@@ -20,6 +20,6 @@
       <state_interface name="effort" />
     </joint>
-    <xacro:include filename="$(find tiago_description)/urdf/head/head.transmission.xacro" />
-    <xacro:head_transmission name="${name}" reduction="${reduction}" offset_value="${offset}"/>
+    <xacro:include filename="$(find tiago_description)/ros2_control/transmissions.urdf.xacro" />
+    <xacro:tiago_simple_transmission name="${name}" reduction="${reduction}" offset_value="${offset}" />
   </xacro:macro>
 </robot>

File: tiago_description/urdf/head/head.urdf.xacro (robot description, xacro)
@@ -15,5 +15,4 @@
   <!--File includes-->
   <xacro:include filename="$(find tiago_description)/urdf/deg_to_rad.xacro" />
-  <xacro:include filename="$(find tiago_description)/urdf/head/head.transmission.xacro" />
   <xacro:include filename="$(find tiago_description)/urdf/sensors/xtion_pro_live.urdf.xacro" />
   <xacro:include filename="$(find tiago_description)/urdf/sensors/orbbec_astra.urdf.xacro" />
@@ -72,6 +71,4 @@
        <implicitSpringDamper>1</implicitSpringDamper>
     </gazebo>
-    <!-- extensions -->
-    <xacro:head_transmission name="${name}" reduction="1" offset_value="${head_1_joint_offset}"/>
   </xacro:macro>
   <!--************************-->
@@ -113,5 +110,4 @@
                          soft_upper_limit="${head_2_upper_limit * deg_to_rad - head_eps}" />
     </joint>
-    <xacro:head_transmission name="${name}" reduction="1" offset_value="${head_2_joint_offset}"/>
   </xacro:macro>
   <xacro:macro name="head" params="name parent camera_model description_calibration_dir extrinsic_calibration_dir no_safety_eps:=False">

File: tiago_description/urdf/torso/torso.ros2_control.xacro (robot description, xacro)
@@ -20,6 +20,6 @@
       <state_interface name="effort" />
     </joint>
-    <xacro:include filename="$(find tiago_description)/urdf/torso/torso.transmission.xacro" />
-    <xacro:torso_simple_transmission name="${name}" reduction="${reduction}" />
+    <xacro:include filename="$(find tiago_description)/ros2_control/transmissions.urdf.xacro" />
+    <xacro:tiago_simple_transmission name="${name}" reduction="${reduction}" />
   </xacro:macro>
 </robot>

File: tiago_description/urdf/torso/torso.urdf.xacro (robot description, xacro)
@@ -15,5 +15,4 @@
   <!--File includes-->
   <xacro:include filename="$(find tiago_description)/urdf/deg_to_rad.xacro" />
-  <xacro:include filename="$(find tiago_description)/urdf/torso/torso.transmission.xacro" />
   <!--Constant parameters-->
   <xacro:property name="torso_max_vel"  value="0.07" />
