Commit message: Imported upstream version '4.0.27' of 'upstream'

File: tiago_description/robots/tiago.urdf.xacro (robot description, xacro)
@@ -26,5 +26,5 @@
     <xacro:arg name="namespace" default=""/>
     <xacro:arg name="no_safety_eps" default="false"/>
-    <xacro:arg name="use_sim" default="true"/>
+    <xacro:arg name="use_sim" default="false"/>
     <xacro:property name="arm" value="$(arg arm)" />
     <xacro:if value="${arm not in ['right-arm', 'no-arm']}">
@@ -90,5 +90,5 @@
     use_sim="$(arg use_sim)" />
   <!-- Materials for visualization -->
-  <xacro:include filename="$(find tiago_description)/urdf/materials.urdf.xacro" />
+  <xacro:include filename="$(find pal_urdf_utils)/urdf/materials.urdf.xacro" />
   <!-- Now we can start using the macros included above to define the actual robot -->
   <xacro:base_sensors name="base" laser_model="$(arg laser_model)" sonars="true" microphone="true"/>
@@ -107,4 +107,5 @@
   <xacro:if value="${has_ft_sensor}">
       <xacro:ft_sensor name="wrist" parent="arm_tool_link" />
+      <xacro:force_torque_sensor_gazebo name="wrist_ft" update_rate="100"/>
   </xacro:if>
   <!-- Thermal camera -->
@@ -136,6 +137,3 @@
       </inertial>
   </link>
-  <xacro:if value="${has_ft_sensor}">
-    <xacro:force_torque_sensor_gazebo joint_name="wrist_ft_joint" update_rate="100"/>
-  </xacro:if>
 </robot>

File: tiago_description/ros2_control/ros2_control.urdf.xacro (robot description, xacro)
@@ -14,5 +14,5 @@
 <robot xmlns:xacro="http://ros.org/wiki/xacro"
        name="tiago" >
-  <xacro:macro name="tiago_ros2_control" params="use_sim:=^|true">
+  <xacro:macro name="tiago_ros2_control" params="use_sim:=^|false">
     <xacro:arg name="arm" default="true" />
     <xacro:arg name="end_effector" default="pal-hey5"/>
@@ -82,7 +82,5 @@
       <xacro:if value="${has_ft_sensor}">
         <xacro:include filename="$(find tiago_description)/urdf/sensors/sensors.ros2_control.xacro"/>
-        <xacro:if value="$(arg use_sim)">
-          <xacro:ros2_control_force_torque_sensor name="wrist_ft_joint_force_torque"/>
-        </xacro:if>
+        <xacro:ros2_control_force_torque_sensor name="wrist_ft_sensor"/>
       </xacro:if>
     </ros2_control>

File: tiago_description/urdf/arm/arm.urdf.xacro (robot description, xacro)
@@ -14,5 +14,5 @@
 <robot xmlns:xacro="http://ros.org/wiki/xacro">
   <!--File includes-->
-  <xacro:include filename="$(find tiago_description)/urdf/deg_to_rad.xacro" />
+  <xacro:include filename="$(find pal_urdf_utils)/urdf/deg_to_rad.urdf.xacro" />
   <xacro:include filename="$(find tiago_description)/urdf/arm/wrist.urdf.xacro" />
   <!--Constant parameters-->

File: tiago_description/urdf/arm/wrist.urdf.xacro (robot description, xacro)
@@ -14,5 +14,5 @@
 <robot xmlns:xacro="http://ros.org/wiki/xacro">
   <!--File includes-->
-  <xacro:include filename="$(find tiago_description)/urdf/deg_to_rad.xacro" />
+  <xacro:include filename="$(find pal_urdf_utils)/urdf/deg_to_rad.urdf.xacro" />
   <!--Constant parameters-->
   <xacro:property name="wrist_friction"       value="1.0" />

File: tiago_description/urdf/calibration/calibration_constants.urdf.xacro (robot description, xacro)
@@ -14,5 +14,5 @@
 <robot xmlns:xacro="http://ros.org/wiki/xacro">
   <!--File includes-->
-  <xacro:include filename="$(find tiago_description)/urdf/deg_to_rad.xacro" />
+  <xacro:include filename="$(find pal_urdf_utils)/urdf/deg_to_rad.urdf.xacro" />
   <!--Constant parameters-->
   <xacro:property name="camera_position_x" value="0.0908" />

File: tiago_description/urdf/calibration/extrinsic_camera_calibration_constants.urdf.xacro (robot description, xacro)
@@ -14,5 +14,5 @@
 <robot xmlns:xacro="http://ros.org/wiki/xacro">
   <!--File includes-->
-  <xacro:include filename="$(find tiago_description)/urdf/deg_to_rad.xacro" />
+  <xacro:include filename="$(find pal_urdf_utils)/urdf/deg_to_rad.urdf.xacro" />
 <xacro:macro name="camera_baseline_constants" params="camera_model" >
   <xacro:if value="${camera_model == 'orbbec-astra'}">

File: tiago_description/urdf/end_effector/end_effector.urdf.xacro (robot description, xacro)
@@ -14,5 +14,5 @@
 <robot xmlns:xacro="http://ros.org/wiki/xacro">
   <!--File includes-->
-  <xacro:include filename="$(find tiago_description)/urdf/deg_to_rad.xacro" />
+  <xacro:include filename="$(find pal_urdf_utils)/urdf/deg_to_rad.urdf.xacro" />
   <xacro:include filename="$(find hey5_description)/urdf/hey5_hand.urdf.xacro" />
   <!--

File: tiago_description/urdf/head/head.urdf.xacro (robot description, xacro)
@@ -14,5 +14,5 @@
 <robot xmlns:xacro="http://ros.org/wiki/xacro">
   <!--File includes-->
-  <xacro:include filename="$(find tiago_description)/urdf/deg_to_rad.xacro" />
+  <xacro:include filename="$(find pal_urdf_utils)/urdf/deg_to_rad.urdf.xacro" />
   <xacro:include filename="$(find tiago_description)/urdf/sensors/xtion_pro_live.urdf.xacro" />
   <xacro:include filename="$(find tiago_description)/urdf/sensors/orbbec_astra.urdf.xacro" />

File: tiago_description/urdf/sensors/ftsensor.gazebo.xacro (robot description, xacro)
@@ -13,8 +13,8 @@
  -->
 <robot xmlns:xacro="http://ros.org/wiki/xacro">
-  <xacro:macro name="force_torque_sensor_gazebo" params="joint_name update_rate">
-  <gazebo reference="${joint_name}">
+  <xacro:macro name="force_torque_sensor_gazebo" params="name update_rate">
+  <gazebo reference="${name}_joint">
     <preserveFixedJoint>true</preserveFixedJoint> <!-- in case this is in a fixed joint -->
-    <sensor name="${joint_name}_force_torque" type="force_torque">
+    <sensor name="${name}_sensor" type="force_torque">
       <update_rate>${update_rate}</update_rate>
       <visualize>true</visualize>

File: tiago_description/urdf/torso/torso.urdf.xacro (robot description, xacro)
@@ -14,5 +14,5 @@
 <robot xmlns:xacro="http://ros.org/wiki/xacro">
   <!--File includes-->
-  <xacro:include filename="$(find tiago_description)/urdf/deg_to_rad.xacro" />
+  <xacro:include filename="$(find pal_urdf_utils)/urdf/deg_to_rad.urdf.xacro" />
   <!--Constant parameters-->
   <xacro:property name="torso_max_vel"  value="0.07" />

Commit message: Imported upstream version '4.1.1' of 'upstream'

File: tiago_description/robots/tiago.urdf.xacro (robot description, xacro)
@@ -14,5 +14,5 @@
 <robot  xmlns:xacro="http://ros.org/wiki/xacro"
         name="tiago" >
-    <xacro:arg name="arm" default="right-arm"/> <!-- right-arm, no-arm -->
+    <xacro:arg name="arm" default="tiago-arm"/> <!-- tiago-arm, no-arm -->
     <xacro:arg name="wrist_model" default="wrist-2010"/>
     <xacro:arg name="end_effector" default="pal-hey5"/> <!-- no-end-effector, pal-gripper, pal-hey5-->
@@ -28,5 +28,5 @@
     <xacro:arg name="use_sim" default="false"/>
     <xacro:property name="arm" value="$(arg arm)" />
-    <xacro:if value="${arm not in ['right-arm', 'no-arm']}">
+    <xacro:if value="${arm not in ['right-arm', 'tiago-arm', 'no-arm']}">
       <xacro:wrong_arm/>
     </xacro:if>
@@ -45,5 +45,5 @@
     </xacro:if>
   </xacro:if>
-  <xacro:if value="${end_effector not in ['no-end-effector', 'pal-gripper', 'pal-hey5', 'custom']}">
+  <xacro:if value="${end_effector not in ['no-end-effector', 'pal-gripper', 'pal-hey5', 'custom', 'robotiq-2f-85', 'robotiq-2f-140']}">
     <xacro:wrong_end_effector/>
   </xacro:if>

File: tiago_description/ros2_control/ros2_control.urdf.xacro (robot description, xacro)
@@ -31,4 +31,7 @@
       <xacro:if value="${end_effector == 'pal-hey5'}">
         <xacro:include filename="$(find pal_hey5_description)/urdf/pal_hey5.ros2_control.xacro" />
+      </xacro:if>
+      <xacro:if value="${end_effector in ['robotiq-2f-85', 'robotiq-2f-140']}">
+        <xacro:include filename="$(find pal_robotiq_description)/urdf/robotiq.ros2_control.xacro" />
       </xacro:if>
     </xacro:if>
@@ -78,4 +81,12 @@
           <xacro:ros2_control_hey5 name="hand"/>
         </xacro:if>
+        <xacro:if value="${end_effector == 'robotiq-2f-85'}">
+          <!-- robotiq-2f-85 -->
+          <xacro:ros2_control_robotiq_85_gripper name="gripper" reduction="1.0" />
+        </xacro:if>
+        <xacro:if value="${end_effector == 'robotiq-2f-140'}">
+          <!-- robotiq-2f-140 -->
+          <xacro:ros2_control_robotiq_140_gripper name="gripper" reduction="1.0" />
+        </xacro:if>
       </xacro:if>
       <!-- Force Torque sensor -->

File: tiago_description/urdf/arm/arm.urdf.xacro (robot description, xacro)
@@ -153,5 +153,5 @@
     <link name="${name}_4_link">
       <inertial>
-        <origin xyz="${reflect * -0.095658} ${reflect * 0.014666} 0.018133" rpy="0.00000 0.00000 0.00000"/>
+        <origin xyz="${reflect * -0.095658} ${reflect * 0.014666} ${reflect * 0.018133}" rpy="0.00000 0.00000 0.00000"/>
         <mass value="1.432697"/>
         <inertia ixx="0.002040" ixy="${reflect * 0.000725}" ixz="${-reflect * 0.001150}"

File: tiago_description/urdf/end_effector/end_effector.urdf.xacro (robot description, xacro)
@@ -23,5 +23,5 @@
     - reflect: Set to 1 for a right end effector, or to -1 for a left end effector
   -->
-  <xacro:macro name="tiago_end_effector" params="name parent type reflect">
+  <xacro:macro name="tiago_end_effector" params="name parent type reflect tiago_dual:=false">
   <!-- PAL Gripper -->
   <xacro:if value="${type == 'pal-gripper'}">
@@ -31,4 +31,25 @@
     </xacro:pal_gripper>
   </xacro:if>
+  <!-- Robotiq 2F-85 Gripper -->
+  <xacro:if value="${type == 'robotiq-2f-85'}">
+    <xacro:include filename="$(find pal_robotiq_description)/urdf/robotiq_85_gripper.urdf.xacro" />
+    <xacro:robotiq_85_gripper prefix="${name}_" parent="${parent}" >
+      <origin xyz="0.01 0 0" rpy="${90*deg_to_rad} ${0*deg_to_rad} ${90*deg_to_rad}"/>
+    </xacro:robotiq_85_gripper>
+  </xacro:if>
+  <!-- Robotiq 2F-140 Gripper -->
+  <xacro:if value="${type == 'robotiq-2f-140'}">
+    <xacro:include filename="$(find pal_robotiq_description)/urdf/robotiq_140_gripper.urdf.xacro" />
+    <xacro:robotiq_140_gripper prefix="${name}_" parent="${parent}" >
+      <origin xyz="0.01 0 0" rpy="${90*deg_to_rad} ${0*deg_to_rad} ${90*deg_to_rad}"/>
+    </xacro:robotiq_140_gripper>
+  </xacro:if>
+  <!-- Robotiq Epick Gripper -->
+  <!-- <xacro:if value="${type == 'robotiq-epick'}">
+    <xacro:include filename="$(find pal_robotiq_epick_description)/urdf/robotiq_epick_model_macro.xacro" />
+    <xacro:epick_hand  prefix="${name}_" parent="${parent}">
+      <origin xyz="0.01 0 0" rpy="${90*deg_to_rad} ${0*deg_to_rad} ${90*deg_to_rad}"/>
+    </xacro:epick_hand>
+  </xacro:if> -->
   <!-- Hand -->
   <xacro:if value="${type == 'pal-hey5'}">
@@ -64,10 +85,25 @@
   </xacro:if>
   <!-- Custom -->
-  <!-- <xacro:if value="${type == 'custom'}">
+  <!--xacro:if value="${type == 'custom' and not tiago_dual}">
     <xacro:include filename="$(find custom_ee_description)/urdf/end-effector.urdf.xacro" />
     <xacro:end_effector parent="${parent}">
       <origin xyz="0.01 0 0" rpy="${90*deg_to_rad} ${90*deg_to_rad} ${-90*deg_to_rad}"/>
     </xacro:end_effector>
-  </xacro:if> -->
+  </xacro:if-->
+  <!-- Custom dual-->
+  <!--xacro:if value="${type == 'custom' and tiago_dual}">
+    <xacro:if value="${reflect == 1}"--> <!-- If right -->
+    <!--xacro:include filename="$(find custom_dual_ee_description)/urdf/end-effector-right.urdf.xacro" />
+    <xacro:end_effector_right parent="${parent}">
+      <origin xyz="0.01 0 0" rpy="${90*deg_to_rad} ${90*deg_to_rad} ${-90*deg_to_rad}"/>
+    </xacro:end_effector_right>
+    </xacro:if>
+    <xacro:if value="${reflect == -1}"--> <!-- If left -->
+    <!--xacro:include filename="$(find custom_dual_ee_description)/urdf/end-effector-left.urdf.xacro" />
+    <xacro:end_effector_left parent="${parent}">
+      <origin xyz="0.01 0 0" rpy="${90*deg_to_rad} ${90*deg_to_rad} ${-90*deg_to_rad}"/>
+    </xacro:end_effector_left>
+    </xacro:if>
+  </xacro:if-->
   </xacro:macro>
 </robot>

Commit message: Imported upstream version '4.2.16' of 'upstream'

File: tiago_description/robots/tiago.urdf.xacro (robot description, xacro)
@@ -129,6 +129,4 @@
   <!-- Materials for visualization -->
   <xacro:include filename="$(find pal_urdf_utils)/urdf/materials.urdf.xacro" />
-  <!-- Generic simulator_gazebo plugins -->
-  <xacro:include filename="$(find tiago_description)/gazebo/gazebo.urdf.xacro" />
   <!-- ROS 2 control -->
   <xacro:include filename="$(find tiago_description)/ros2_control/ros2_control.urdf.xacro" />
@@ -136,5 +134,5 @@
   <!-- Base -->
   <xacro:if value="${base_type == 'pmb2'}">
-    <xacro:base_sensors name="base" laser_model="${laser_model}" sonars="true" microphone="true"/>
+    <xacro:base_sensors name="base" laser_model="${laser_model}" has_sonars="true" has_microphone="true"/>
   </xacro:if>
   <xacro:if value="${base_type == 'omni_base'}">

File: tiago_description/ros2_control/ros2_control.urdf.xacro (robot description, xacro)
@@ -42,4 +42,12 @@
   <!-- MACRO DEFINITION-->
   <xacro:macro name="tiago_ros2_control">
+    <!-- Init the ROS 2 control gazebo interface -->
+    <xacro:if value="${use_sim_time}">
+      <gazebo>
+        <plugin filename="libgazebo_ros2_control.so" name="gazebo_ros2_control">
+          <parameters>$(find tiago_description)/ros2_control/gazebo_controller_manager_cfg.yaml</parameters>
+        </plugin>
+      </gazebo>
+    </xacro:if>
     <!-- ROS 2 control config-->
     <ros2_control name="ros2_control_tiago_system" type="system">
@@ -48,4 +56,6 @@
         <xacro:if value="${use_sim_time}">
           <plugin>gazebo_ros2_control/GazeboSystem</plugin>
+        <!-- IMU sensor (only in simulation)-->
+        <xacro:ros2_control_imu name="base_imu_sensor"/>
         </xacro:if>
         <xacro:unless value="${use_sim_time}">

File: tiago_description/urdf/head/head.urdf.xacro (robot description, xacro)
@@ -109,5 +109,5 @@
     <!-- Asus Xtion-->
     <xacro:if value="${camera_model == 'asus-xtion'}">
-      <xacro:xtion_pro_live name="head_front_camera" parent="${name}_2" camera_model="${camera_model}" extrinsic_calibration_dir="${extrinsic_calibration_dir}">
+      <xacro:xtion_pro_live name="head_front_camera" parent="${name}_2_link" camera_model="${camera_model}" extrinsic_calibration_dir="${extrinsic_calibration_dir}">
         <origin xyz="${camera_position_x} ${camera_position_y} ${camera_position_z}" rpy="${camera_orientation_r} ${camera_orientation_p} ${camera_orientation_y}" />
         <!-- optical origin -->
@@ -117,5 +117,5 @@
     <!-- Orbecc Astra-->
     <xacro:if value="${camera_model in ['orbbec-astra', 'orbbec-astra-pro']}">
-      <xacro:orbbec_astra name="head_front_camera" parent="${name}_2" camera_model="${camera_model}" extrinsic_calibration_dir="${extrinsic_calibration_dir}">
+      <xacro:orbbec_astra name="head_front_camera" parent="${name}_2_link" camera_model="${camera_model}" extrinsic_calibration_dir="${extrinsic_calibration_dir}">
         <origin xyz="${camera_position_x} ${camera_position_y} ${camera_position_z}" rpy="${camera_orientation_r} ${camera_orientation_p} ${camera_orientation_y}" />
         <!-- optical origin -->

File: tiago_description/urdf/sensors/orbbec_astra.urdf.xacro (robot description, xacro)
@@ -22,5 +22,5 @@
     <joint name="${name}_joint" type="fixed">
       <xacro:insert_block name="origin"/>
-      <parent link="${parent}_link"/>
+      <parent link="${parent}"/>
       <child link="${name}_link"/>
     </joint>

File: tiago_description/urdf/sensors/xtion_pro_live.urdf.xacro (robot description, xacro)
@@ -21,5 +21,5 @@
     <joint name="${name}_joint" type="fixed">
       <xacro:insert_block name="origin"/>
-      <parent link="${parent}_link"/>
+      <parent link="${parent}"/>
       <child link="${name}_link"/>
     </joint>

Commit message: Imported upstream version '4.6.0' of 'upstream'

File: tiago_description/robots/tiago.urdf.xacro (robot description, xacro)
@@ -34,5 +34,5 @@
   <xacro:arg name="ft_sensor" default="schunk-ft"/>
   <!-- wrist-2010, wrist-2017 -->
-  <xacro:arg name="wrist_model" default="wrist-2010"/>
+  <xacro:arg name="wrist_model" default="wrist-2017"/>
   <!-- no-end-effector, pal-gripper, pal-hey5, custom, robotiq-2f-85,robotiq-2f-140-->
   <xacro:arg name="end_effector" default="pal-hey5"/>
@@ -140,5 +140,12 @@
   </xacro:if>
   <!-- Torso -->
-  <xacro:tiago_torso name="torso" parent="base_link"/>
+  <xacro:tiago_torso name="torso" parent="base_link">
+    <xacro:if value="${base_type == 'pmb2'}">
+      <origin rpy="0 0 0" xyz="-0.062 0.0 0.193" />
+    </xacro:if>
+    <xacro:if value="${base_type == 'omni_base'}">
+      <origin rpy="0 0 0" xyz="-0.062 0.0 0.215" />
+    </xacro:if>
+  </xacro:tiago_torso>
   <!-- Arm, FT, EE -->
   <xacro:if value="${has_arm}">

File: tiago_description/urdf/arm/arm.urdf.xacro (robot description, xacro)
@@ -32,8 +32,8 @@
     <!-- Param related properties -->
     <xacro:if value="${wrist_model == 'wrist-2010'}">
-      <xacro:property name="tool_link_z_offset" value="0.046"/>
+      <xacro:property name="tool_link_z_offset" value="${ 0.056873 if has_ft_sensor else 0.0518 }"/>
     </xacro:if>
     <xacro:if value="${wrist_model == 'wrist-2017'}">
-      <xacro:property name="tool_link_z_offset" value="${ 0.046 if has_ft_sensor else 0.0573 }"/>
+      <xacro:property name="tool_link_z_offset" value="${ 0.051875 if has_ft_sensor else 0.0615 }"/>
     </xacro:if>
     <!-- Shoulder -->

File: tiago_description/urdf/sensors/ftsensor.urdf.xacro (robot description, xacro)
@@ -20,6 +20,6 @@
     <link name="${name}_ft_link">
       <inertial>
-        <mass value="0.1" />
-        <inertia ixx="0.0" ixy="0.0" ixz="0.0" iyy="0.0" iyz="0.0" izz="0.0" />
+        <mass value="0.095000" />
+        <inertia ixx="0.000016" ixy="-0.000001" ixz="0.0" iyy="0.000015" iyz="0.0" izz="0.000027" />
       </inertial>
       <visual>
@@ -40,5 +40,5 @@
       <parent link="${parent}" />
       <child link="${name}_ft_link" />
-      <origin xyz="${0.0157*0.5} 0 0" rpy="${90.0 * deg_to_rad} 0 ${90.0 * deg_to_rad}" />
+      <origin xyz="${0.0157*0.5 + 0.001525} 0 0" rpy="${90.0 * deg_to_rad} 0 ${90.0 * deg_to_rad}" />
     </joint>
     <!-- FT tool -->
@@ -65,5 +65,5 @@
       <parent link="${name}_ft_link" />
       <child link="${name}_ft_tool_link" />
-      <origin xyz="0 0 ${0.0157*0.5 + 0.00975*0.5}" rpy="${-90.0 * deg_to_rad} ${-90.0 * deg_to_rad} 0" />
+      <origin xyz="0 0 ${0.0157*0.5 + 0.00975*0.5 - 0.001525}" rpy="${-90.0 * deg_to_rad} ${-90.0 * deg_to_rad} 0" />
     </joint>
     <!-- Gazebo config-->

File: tiago_description/urdf/torso/torso.urdf.xacro (robot description, xacro)
@@ -19,5 +19,5 @@
   <xacro:include filename="$(find pal_urdf_utils)/urdf/deg_to_rad.urdf.xacro" />
   <!-- MACRO DEFINITION-->
-  <xacro:macro name="tiago_torso" params="name parent">
+  <xacro:macro name="tiago_torso" params="name parent *origin">
     <!-- Bottom fixed part of column -->
     <link name="${name}_fixed_link">
@@ -48,5 +48,5 @@
     </link>
     <joint name="${name}_fixed_joint" type="fixed">
-      <origin rpy="0 0 0" xyz="-0.062 0.0 0.193" />
+      <xacro:insert_block name="origin"/>
       <parent link="${parent}" />
       <child link="${name}_fixed_link" />
@@ -79,5 +79,5 @@
     </gazebo>
     <joint name="${name}_fixed_column_joint" type="fixed">
-      <origin rpy="0 0 0" xyz="-0.062 0 0.195" />
+      <xacro:insert_block name="origin"/>
       <parent link="${parent}" />
       <child link="${name}_fixed_column_link" />
